Commit message: add datalayer type as well in urdf

File: datalayer_bringup/urdf/datalayer_hardware_interface_nrt.ros2_control.xacro (robot description, xacro)
@@ -6,4 +6,7 @@
       <hardware>
         <plugin>datalayer_hardware_interface/DataLayerHardwareInterface_NRT</plugin>
+        <param name="device_ip">127.0.0.1</param>
+        <param name="device_user">boschrexroth</param>
+        <param name="device_password">boschrexroth</param>
       </hardware>
       <!--Addresses MUST ommit stating and ending backslash-->
@@ -11,6 +14,6 @@
         <xacro:state_interface_DataLayer_NRT
           name="scheduler_counter" DL_address="scheduler/admin/info/common-data-rt" DL_variable="counter"/>
-        <xacro:comand_interface_DataLayer_NRT initial_value="1.0"
-          name="ping_timeout" DL_address="datalayer/server/settings" DL_variable="​serverIdlePingTimeout​"/>
+        <!-- <xacro:comand_interface_DataLayer_NRT initial_value="1.0"
+          name="ping_timeout" DL_address="datalayer/server/settings" DL_variable="​serverIdlePingTimeout​"/> -->
       </gpio>
     </ros2_control>

File: datalayer_bringup/urdf/datalayer_interfaces.ros2_control.xacro (robot description, xacro)
@@ -2,11 +2,12 @@
 <robot xmlns:xacro="http://wiki.ros.org/xacro">
     <!--Addresses MUST ommit stating and ending backslash-->
-    <xacro:macro name="state_interface_DataLayer_NRT" params="name DL_address DL_variable">
+    <xacro:macro name="state_interface_DataLayer_NRT" params="name DL_address DL_variable DL_variable_type">
         <state_interface name="${name}">
             <param name="DL_address">${DL_address}</param>
             <param name="DL_variable">${DL_variable}</param>
+            <param name="DL_variable_type">${DL_variable_type}</param>
         </state_interface>
     </xacro:macro>
-    <xacro:macro name="command_interface_DataLayer_NRT" params="name initial_value:='' DL_address DL_variable">
+    <xacro:macro name="command_interface_DataLayer_NRT" params="name initial_value:='' DL_address DL_variable DL_variable_type">
         <command_interface name="${name}">
             <xacro:if value="${initial_value != ''}">
@@ -15,4 +16,5 @@
             <param name="DL_address">${DL_address}</param>
             <param name="DL_variable">${DL_variable}</param>
+            <param name="DL_variable_type">${DL_variable_type}</param>
         </command_interface>
     </xacro:macro>
